File: pcb/lighthouse-pcb.kicad_pcb (KiCad board)
At the start: 2 copper layers, 45 x 45 mm, 50 parts, among them J1 USB_C_Receptacle_USB2.0, SW1 BOOT/ROOF, SW3 FRONT, SW4 SW_DIP_x08, U1 ESP32-C3-WROOM-02, U2 CN5711, U3 AP2112K-3.3, U4 USBLC6-2SC6

Commit message: Remove tooling hole
Parts:
- removed H1, H2, H3: JLCPCB tooling hole, lighthouse_footprints:JLCPCB tooling hole
Other:
- board text removed: "JLCJLCJLCJLC"

Commit message: Add information for panelization
Parts:
- added T1: Tab, PCM_kikit:Tab, F.Cu at (100.0, 55.0)
- added T2: Tab, PCM_kikit:Tab, F.Cu at (100.0, 90.0)
- added T3: Tab, PCM_kikit:Tab, F.Cu at (145.0, 55.0)
- added T4: Tab, PCM_kikit:Tab, F.Cu at (145.0, 90.0)
